File: FT03/ft03.kicad_pcb (KiCad board)
At the start: 4 copper layers, 40.9 x 23.7 mm, 89 parts, among them J1 UART, Q1 SNM2308S, Q10 CJE3139K, Q11 DTC143E, Q2 SNM2308S, Q3 SNM2308S, Q5 DTC143E, Q6 DTC143E, Q7 DTC143E, Q8 DTC143E, Q9 CJE3139K, U1 CS32F031K8V6, U2 M25PX32-VMP, U3 LDO, U4 PC3221, U5 LCD, U6 TTP223-BA6

Commit message: LDO regulator p/n
Parts:
- U3: value LDO -> CJ6330A33M
