File: FT03/ft03.kicad_sch (KiCad schematic)
At the start: 89 parts, among them J1 UART, Q1 SNM2308S, Q10 CJE3139K, Q11 DTC143E, Q2 SNM2308S, Q3 SNM2308S, Q5 DTC143E, Q6 DTC143E, Q7 DTC143E, Q8 DTC143E, Q9 CJE3139K, U1 CS32F031K8V6, U2 M25PX32-VMP, U3 LDO, U4 PC3221, U5 LCD, U6 TTP223-BA6

Commit message: LDO regulator p/n
Parts:
- removed U3: LDO, Active:SOT95P230X117-3, symbol Connector_Generic:Conn_01x03
- added U3: CJ6330A33M, Active:SOT95P230X117-3, symbol Regulator_Linear:AP2127N3-1.2
Connections:
- net +3V3: now also U3.2 (VO)
- net +BATT: now also U3.3 (VI)
- net GND: now also U3.1 (GND)
Other:
- moved on the sheet: TP16
Changed lines of the file:
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@@
 	)
 	(junction
-		(at 215.9 40.64)
+		(at 207.01 27.94)
 		(diameter 0)
 		(color 0 0 0 0)
@@
 	(wire
 		(pts
-			(xy 215.9 38.1) (xy 215.9 40.64)
+			(xy 207.01 25.4) (xy 207.01 27.94)
 		)
 		(stroke
@@
 	(wire
 		(pts
-			(xy 223.52 38.1) (xy 219.71 38.1)
-		)
-		(stroke
-			(width 0)
-			(type default)
-		)
-	)
-	(wire
-		(pts
 			(xy 193.04 123.19) (xy 200.66 123.19)
 		)
@@
 	(wire
 		(pts
-			(xy 222.25 35.56) (xy 222.25 43.18)
-		)
-		(stroke
-			(width 0)
-			(type default)
-		)
-	)
-	(wire
-		(pts
 			(xy 87.63 109.22) (xy 100.33 109.22)
 		)
@@
 	(wire
 		(pts
+			(xy 226.06 27.94) (xy 228.6 27.94)
+		)
+		(stroke
+			(width 0)
+			(type default)
+		)
+	)
+	(wire
+		(pts
 			(xy 256.54 140.97) (xy 256.54 144.78)
 		)
@@
 	(wire
 		(pts
-			(xy 223.52 35.56) (xy 222.25 35.56)
-		)
-		(stroke
-			(width 0)
-			(type default)
-		)
-	)
-	(wire
-		(pts
 			(xy 76.2 96.52) (xy 100.33 96.52)
 		)
@@
 	(wire
 		(pts
-			(xy 219.71 33.02) (xy 219.71 38.1)
-		)
-		(stroke
-			(width 0)
-			(type default)
-		)
-	)
-	(wire
-		(pts
 			(xy 246.38 25.4) (xy 246.38 27.94)
 		)
@@
 	(wire
 		(pts
-			(xy 215.9 40.64) (xy 223.52 40.64)
+			(xy 207.01 27.94) (xy 210.82 27.94)
 		)
 		(stroke
@@
 	(wire
 		(pts
+			(xy 228.6 26.67) (xy 228.6 27.94)
+		)
+		(stroke
+			(width 0)
+			(type default)
+		)
+	)
+	(wire
+		(pts
 			(xy 137.16 34.29) (xy 137.16 35.56)
 		)
@@
 	(symbol
 		(lib_id "power:+BATT")
-		(at 215.9 38.1 0)
+		(at 207.01 25.4 0)
 		(unit 1)
 		(exclude_from_sim no)
@@
 		(fields_autoplaced yes)
 		(property "Reference" "#PWR018"
-			(at 215.9 41.91 0)
+			(at 207.01 29.21 0)
 			(effects
 				(font
@@
 		)
 		(property "Value" "+BATT"
-			(at 215.9 33.02 0)
+			(at 207.01 20.32 0)
 			(effects
 				(font
@@
 		)
 		(property "Footprint" ""
-			(at 215.9 38.1 0)
+			(at 207.01 25.4 0)
 			(effects
 				(font
@@
 		)
 		(property "Datasheet" ""
-			(at 215.9 38.1 0)
+			(at 207.01 25.4 0)
 			(effects
 				(font
@@
 		)
 		(property "Description" "Power symbol creates a global label with name \"+BATT\""
-			(at 215.9 38.1 0)
+			(at 207.01 25.4 0)
 			(effects
 				(font
@@
 	(symbol
 		(lib_id "power:GND")
-		(at 222.25 43.18 0)
+		(at 218.44 35.56 0)
 		(unit 1)
 		(exclude_from_sim no)
@@
 		(fields_autoplaced yes)
 		(property "Reference" "#PWR042"
-			(at 222.25 49.53 0)
+			(at 218.44 41.91 0)
 			(effects
 				(font
@@
 		)
 		(property "Value" "GND"
-			(at 222.25 49.53 0)
+			(at 218.44 41.91 0)
 			(effects
 				(font
@@
 		)
 		(property "Footprint" ""
-			(at 222.25 43.18 0)
+			(at 218.44 35.56 0)
 			(effects
 				(font
@@
 		)
 		(property "Datasheet" ""
-			(at 222.25 43.18 0)
+			(at 218.44 35.56 0)
 			(effects
 				(font
@@
 		)
 		(property "Description" "Power symbol creates a global label with name \"GND\" , ground"
-			(at 222.25 43.18 0)
+			(at 218.44 35.56 0)
 			(effects
 				(font
@@
 	)
 	(symbol
-		(lib_id "Connector_Generic:Conn_01x03")
-		(at 228.6 38.1 0)
-		(unit 1)
-		(exclude_from_sim no)
-		(in_bom yes)
-		(on_board yes)
-		(dnp no)
-		(fields_autoplaced yes)
-		(property "Reference" "U3"
-			(at 231.14 36.8299 0)
-			(effects
-				(font
-					(size 1.27 1.27)
-				)
-				(justify left)
-			)
-		)
-		(property "Value" "LDO"
-			(at 231.14 39.3699 0)
-			(effects
-				(font
-					(size 1.27 1.27)
-				)
-				(justify left)
-			)
-		)
-		(property "Footprint" "Active:SOT95P230X117-3"
-			(at 228.6 38.1 0)
-			(effects
-				(font
-					(size 1.27 1.27)
-				)
-				(hide yes)
-			)
-		)
-		(property "Datasheet" "~"
-			(at 228.6 38.1 0)
-			(effects
-				(font
-					(size 1.27 1.27)
-				)
-				(hide yes)
-			)
-		)
-		(property "Description" "Generic connector, single row, 01x03, script generated (kicad-library-utils/schlib/autogen/connector/)"
-			(at 228.6 38.1 0)
-			(effects
-				(font
-					(size 1.27 1.27)
-				)
-				(hide yes)
-			)
-		)
-		(property "Topmark" "A7y49"
-			(at 228.6 38.1 0)
-			(effects
-				(font
-					(size 1.27 1.27)
-				)
-				(hide yes)
-			)
-		)
-		(pin "1"
-		)
-		(pin "3"
-		)
-		(pin "2"
-		)
-		(instances
-			(project ""
-				(path "/059f7830-59f0-44e4-9b75-0a4f04ba074b"
-					(reference "U3")
-					(unit 1)
-				)
-			)
-		)
-	)
-	(symbol
 		(lib_id "power:GND")
 		(at 76.2 102.87 0)
@@
 	(symbol
 		(lib_id "power:+3V3")
-		(at 219.71 33.02 0)
+		(at 228.6 26.67 0)
 		(unit 1)
 		(exclude_from_sim no)
@@
 		(fields_autoplaced yes)
 		(property "Reference" "#PWR039"
-			(at 219.71 36.83 0)
+			(at 228.6 30.48 0)
 			(effects
 				(font
@@
 		)
 		(property "Value" "+3V3"
-			(at 219.71 27.94 0)
+			(at 228.6 21.59 0)
 			(effects
 				(font
@@
 		)
 		(property "Footprint" ""
-			(at 219.71 33.02 0)
+			(at 228.6 26.67 0)
 			(effects
 				(font
@@
 		)
 		(property "Datasheet" ""
-			(at 219.71 33.02 0)
+			(at 228.6 26.67 0)
 			(effects
 				(font
@@
 		)
 		(property "Description" "Power symbol creates a global label with name \"+3V3\""
-			(at 219.71 33.02 0)
+			(at 228.6 26.67 0)
 			(effects
 				(font
@@
 	(symbol
 		(lib_id "Connector:TestPoint")
-		(at 215.9 40.64 90)
+		(at 207.01 27.94 90)
 		(unit 1)
 		(exclude_from_sim no)
@@
 		(fields_autoplaced yes)
 		(property "Reference" "TP16"
-			(at 212.598 35.56 90)
+			(at 203.708 22.86 90)
 			(effects
 				(font
@@
 		)
 		(property "Value" "B+"
-			(at 212.598 38.1 90)
+			(at 203.708 25.4 90)
 			(effects
 				(font
@@
 		)
 		(property "Footprint" "TestPoint:TestPoint_Pad_D1.5mm"
-			(at 215.9 35.56 0)
+			(at 207.01 22.86 0)
 			(effects
 				(font
@@
 		)
 		(property "Datasheet" "~"
-			(at 215.9 35.56 0)
+			(at 207.01 22.86 0)
 			(effects
 				(font
@@
 		)
 		(property "Description" "test point"
-			(at 215.9 40.64 0)
+			(at 207.01 27.94 0)
 			(effects
 				(font
@@
 					(unit 1)
 				)
+			)
+		)
+	)
+	(symbol
+		(lib_id "Regulator_Linear:AP2127N3-1.2")
+		(at 218.44 27.94 0)
+		(unit 1)
+		(exclude_from_sim no)
+		(in_bom yes)
+		(on_board yes)
+		(dnp no)
+		(property "Reference" "U3"
+			(at 218.44 21.844 0)
+			(effects
+				(font
+					(size 1.27 1.27)
+				)
+			)
+		)
+		(property "Value" "CJ6330A33M"
+			(at 218.44 24.13 0)
+			(effects
+				(font
+					(size 1.27 1.27)
+				)
+			)
+		)
+		(property "Footprint" "Active:SOT95P230X117-3"
+			(at 218.44 22.225 0)
+			(effects
+				(font
+					(size 1.27 1.27)
+					(italic yes)
+				)
+				(hide yes)
+			)
+		)
+		(property "Datasheet" ""
+			(at 218.44 27.94 0)
+			(effects
+				(font
+					(size 1.27 1.27)
+				)
+				(hide yes)
+			)
+		)
+		(property "Description" ""
+			(at 218.44 27.94 0)
+			(effects
+				(font
+					(size 1.27 1.27)
+				)
+				(hide yes)
+			)
+		)
+		(property "Topmark" "A7y49"
+			(at 218.44 27.94 0)
+			(effects
+				(font
+					(size 1.27 1.27)
+				)
+				(hide yes)
+			)
+		)
+		(pin "3"
+		)
+		(pin "1"
+		)
+		(pin "2"
+		)
+		(instances
+			(project ""
+				(path "/059f7830-59f0-44e4-9b75-0a4f04ba074b"
+					(reference "U3")
+					(unit 1)
+				)
