File: YK761/YK761.kicad_pcb (KiCad board)
At the start: 4 copper layers, 34.9 x 20.3 mm, 92 parts, among them J1 LCD+LED, J2 Conn_01x01, J3 Conn_01x01, J4 Conn_01x01, Q1 AP20P01BF, Q2 DTC114E, Q3 DTC114E, Q4 CJE3139K, U1 CST4056, U2 RF01, U3 ?, U4 LDO, U5 Conn_02x03_Counter_Clockwise, Y1 32MHz

Commit message: Add values
Parts:
- removed C21, C22: ?, Capacitor_SMD:C_0402_1005Metric
- added L1: 2uH, Inductor_SMD:L_0402_1005Metric, B.Cu at (148.3, 99.0)
- added L2: 2uH, Inductor_SMD:L_0402_1005Metric, B.Cu at (146.6, 99.7)
- C1, C14, C16: value ? -> 1uF
- C10, C9: value ? -> 10uF
- C11, C15, C18, C24, C4, C5, C7: value ? -> 0.1uF
- C12, C13: value ? -> 12pF
- C17, C2, C3: value ? -> 4.7uF
- C19: value ? -> 470pF
- C20: value ? -> 12.5pF
- C23: value ? -> 2.2uF
- C6: value ? -> 0.01uF
- C8: value ? -> 100pF
- R10, R14, R8, R9: value ? -> 100K
- R11: value ? -> 4.7
- R13, R16: value ? -> 5.1K
- R15: value ? -> 100
- R17: value ? -> 2M
- R18: value ? -> 1M
- R19: value ? -> 1.2K
- R20: value ? -> 3.01K
- R3, R4, R5: value ? -> 10K
- R6: value ? -> 1K
Connections:
- net /P01/SWD renamed /CHG_STDY
- net /P08 renamed /~{BL_ON}
- net /P11 renamed /CHG_EN
- net /P16 renamed /M_ON
- net /P20 renamed /O1_2_ON
- net /P23 renamed /MON_O2
- net /P30 renamed /MON_O1

Commit message: Complete YK761
Parts:
- added C21: 4.7uF, Capacitor_SMD:C_0402_1005Metric, F.Cu at (160.7, 44.3)
- added C22: 4.7uF, Capacitor_SMD:C_0402_1005Metric, F.Cu at (158.4, 41.7)
- added D10: WHT, LED_SMD:LED_0603_1608Metric, F.Cu at (145.3, 15.4)
- added D11: WHT, LED_SMD:LED_0603_1608Metric, F.Cu at (139.8, 15.4)
- added D12: WHT, LED_SMD:LED_0603_1608Metric, F.Cu at (133.3, 16.9)
- added D13: WHT, LED_SMD:LED_0603_1608Metric, F.Cu at (136.9, 19.1)
- added D14: WHT, LED_SMD:LED_0603_1608Metric, F.Cu at (132.6, 25.3)
- added D15: WHT, LED_SMD:LED_0603_1608Metric, F.Cu at (137.2, 26.1)
- added D16: WHT, LED_SMD:LED_0603_1608Metric, F.Cu at (140.9, 23.8)
- added D17: WHT, LED_SMD:LED_0603_1608Metric, F.Cu at (146.4, 25.9)
- added D18: WHT, LED_SMD:LED_0603_1608Metric, F.Cu at (150.8, 25.9)
- added D19: WHT, LED_SMD:LED_0603_1608Metric, F.Cu at (155.8, 23.8)
- added D20: WHT, LED_SMD:LED_0603_1608Metric, F.Cu at (134.7, 22.4)
- added D21: WHT, LED_SMD:LED_0603_1608Metric, F.Cu at (153.6, 16.0)
- added D22: WHT, LED_SMD:LED_0603_1608Metric, F.Cu at (141.5, 26.2)
- added D23: LED_ARGB, LED_SMD:LED_LiteOn_LTST-C295K_1.6x0.8mm, F.Cu at (140.2, 20.4)
- added D24: LED_ARGB, LED_SMD:LED_LiteOn_LTST-C295K_1.6x0.8mm, F.Cu at (143.8, 20.4)
- added D25: LED_ARGB, LED_SMD:LED_LiteOn_LTST-C295K_1.6x0.8mm, F.Cu at (147.6, 20.4)
- added D26: LED_ARGB, LED_SMD:LED_LiteOn_LTST-C295K_1.6x0.8mm, F.Cu at (151.3, 20.4)
- added D4: WHT, LED_SMD:LED_0603_1608Metric, F.Cu at (158.1, 27.3)
- added D5: WHT, LED_SMD:LED_0603_1608Metric, F.Cu at (160.6, 21.6)
- added D6: WHT, LED_SMD:LED_0603_1608Metric, F.Cu at (156.4, 20.0)
- added D7: WHT, LED_SMD:LED_0603_1608Metric, F.Cu at (157.9, 15.7)
- added D8: WHT, LED_SMD:LED_0603_1608Metric, F.Cu at (153.1, 13.6)
- added D9: WHT, LED_SMD:LED_0603_1608Metric, F.Cu at (149.8, 15.4)
- added J10: FLEX, VapeRE:UNK_FPC_1x16-1MP_P0.5mm_Flex, F.Cu at (149.4, 78.7)
- added J5: LCD, VapeRE:UNK_FPC_1x08-1MP_P0.5mm_Horizontal, F.Cu at (161.4, 54.0)
- added Q10: DTC114E, Package_TO_SOT_SMD:SOT-523, F.Cu at (162.6, 41.8)
- added R22: 100, Resistor_SMD:R_0402_1005Metric, F.Cu at (160.1, 26.5)
- added R23: 100, Resistor_SMD:R_0402_1005Metric, F.Cu at (161.0, 18.8)
- added R24: 100, Resistor_SMD:R_0402_1005Metric, F.Cu at (157.6, 18.3)
- added R25: 100, Resistor_SMD:R_0402_1005Metric, F.Cu at (161.0, 15.7)
- added R26: 100, Resistor_SMD:R_0402_1005Metric, F.Cu at (156.7, 13.6)
- added R27: 100, Resistor_SMD:R_0402_1005Metric, F.Cu at (148.0, 14.6)
- added R28: 100, Resistor_SMD:R_0402_1005Metric, F.Cu at (143.6, 14.6)
- added R29: 100, Resistor_SMD:R_0402_1005Metric, F.Cu at (141.6, 14.6)
- added R30: 100, Resistor_SMD:R_0402_1005Metric, F.Cu at (135.1, 16.2)
- added R31: 100, Resistor_SMD:R_0402_1005Metric, F.Cu at (135.6, 18.3)
- added R32: 100, Resistor_SMD:R_0402_1005Metric, F.Cu at (133.3, 27.4)
- added R33: 100, Resistor_SMD:R_0402_1005Metric, F.Cu at (138.5, 26.5)
- added R34: 100, Resistor_SMD:R_0402_1005Metric, F.Cu at (144.8, 23.8)
- added R35: 100, Resistor_SMD:R_0402_1005Metric, F.Cu at (148.1, 26.6)
- added R36: 100, Resistor_SMD:R_0402_1005Metric, F.Cu at (149.3, 26.6)
- added R37: 100, Resistor_SMD:R_0402_1005Metric, F.Cu at (161.2, 36.1)
- added R38: 100, Resistor_SMD:R_0402_1005Metric, F.Cu at (161.3, 39.5)
- added R39: 100, Resistor_SMD:R_0402_1005Metric, F.Cu at (160.0, 36.1)
- added R40: 100, Resistor_SMD:R_0402_1005Metric, F.Cu at (160.1, 39.5)
- added R41: 511, Resistor_SMD:R_0402_1005Metric, F.Cu at (156.2, 36.0)
- added R42: 267, Resistor_SMD:R_0402_1005Metric, F.Cu at (157.5, 36.1)
- added R43: 330, Resistor_SMD:R_0402_1005Metric, F.Cu at (158.7, 36.1)
- added U10: LDO, Active:SOT95P230X117-3, F.Cu at (158.4, 44.1)
Connections:
- net /P03 renamed /LED_BLU
- net /P05 renamed /LED_GRN
- net /P12 renamed /LED_RED
- net /P13 renamed /LED_WH1
- net /P21 renamed /LED_WH2
- net /P22 renamed /LED_WHT
- net Net-(J1-Pin_9) renamed /BACKLIGHT
- net Net-(U2-VDD_1V8) renamed +1V8
Routing:
- net Net-(Q10-C): track 0.00 -> 124.6 mm, vias 0 -> 3
- net /3V3: track 0.00 -> 73.3 mm, vias 0 -> 7
- net Net-(J10-Pin_7): track 0.00 -> 51.7 mm
- net Net-(J10-Pin_12): track 0.00 -> 51.2 mm, vias 0 -> 2
- net Net-(J10-Pin_11): track 0.00 -> 51.2 mm, vias 0 -> 2
- net Net-(J10-Pin_14): track 0.00 -> 50.7 mm, vias 0 -> 2
- net Net-(J10-Pin_13): track 0.00 -> 50.5 mm, vias 0 -> 2
- net Net-(J10-Pin_15): track 0.00 -> 50.4 mm, vias 0 -> 2
- net Net-(J10-Pin_10): track 0.00 -> 47.5 mm, vias 0 -> 2
- net Net-(D20-K): track 0.00 -> 42.4 mm
- net Net-(J10-Pin_16): track 0.00 -> 41.3 mm
- net Net-(D23-GK): track 0.00 -> 34.6 mm
- net Net-(J10-Pin_9): track 0.00 -> 32.5 mm
- net Net-(D23-RK): track 0.00 -> 32.1 mm, vias 0 -> 5
- net Net-(D23-BK): track 0.00 -> 31.9 mm
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- added copper zone on B.Cu, net /3V3
- added copper zone on F.Cu, net /3V3
- added copper zone on F.Cu, net Net-(J10-Pin_6)
- added copper zone on F.Cu, net Net-(J10-Pin_7)

Commit message: LDO regulator p/n
Parts:
- U2: value RF01 -> BLueX Micro RF01 / BX2400
- U3: value ? -> PD64SH4AD
- U4: value LDO -> CJ6330A33M
Connections:
- net /P02 renamed /~{LCD_CS}
- net /P04 renamed /~{LCD_CLK}
- net /P06 renamed /~{LCD_DI}
- net /P07 renamed /~{LCD_RST}
- net /P09 renamed /~{LCD_DC}
- net /~{RESET} renamed /RESET
