File: YK761/YK761.kicad_sch (KiCad schematic)
At the start: 92 parts, among them J1 LCD+LED, J2 Conn_01x01, J3 Conn_01x01, J4 Conn_01x01, Q1 AP20P01BF, Q2 DTC114E, Q3 DTC114E, Q4 CJE3139K, U1 CST4056, U2 RF01, U3 ?, U4 LDO, U5 Conn_02x03_Counter_Clockwise, Y1 32MHz

Commit message: Add values
Parts:
- removed C21, C22: ?, Capacitor_SMD:C_0402_1005Metric, symbol Device:C_Small
- added L1, L2: 2uH, Inductor_SMD:L_0402_1005Metric, symbol Device:L_Small
- C1, C14, C16: value ? -> 1uF
- C10, C9: value ? -> 10uF
- C11, C15, C18, C24, C4, C5, C7: value ? -> 0.1uF
- C12, C13: value ? -> 12pF
- C17, C2, C3: value ? -> 4.7uF
- C19: value ? -> 470pF
- C20: value ? -> 12.5pF
- C23: value ? -> 2.2uF
- C6: value ? -> 0.01uF
- C8: value ? -> 100pF
- R10, R14, R8, R9: value ? -> 100K
- R11: value ? -> 4.7
- R13, R16: value ? -> 5.1K
- R15: value ? -> 100
- R17: value ? -> 2M
- R18: value ? -> 1M
- R19: value ? -> 1.2K
- R20: value ? -> 3.01K
- R3, R4, R5: value ? -> 10K
- R6: value ? -> 1K
Connections:
- net at C10.1, C18.2, U2.17 (VDD_1V8)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: now also L1.1
- net at C20.2: now also L2.2
- net at U2.45 (RF_P): now also L1.2, L2.1
Other:
- moved on the sheet: C17, C2, C24, C3, C5, D2, TP10, TP18, TP9, U4

Commit message: Complete YK761
Parts:
- added C21, C22: 4.7uF, Capacitor_SMD:C_0402_1005Metric, symbol Device:C_Small
- added D10, D11, D12, D13, D14, D15, D16, D17, D18, D19, D20, D21, D22, D4, D5, D6, D7, D8, D9: WHT, LED_SMD:LED_0603_1608Metric, symbol Device:LED_Small_Filled
- added D23, D24, D25, D26: LED_ARGB, LED_SMD:LED_LiteOn_LTST-C295K_1.6x0.8mm, symbol Device:LED_ARGB
- added J10: FLEX, VapeRE:UNK_FPC_1x16-1MP_P0.5mm_Flex, symbol Connector:Conn_01x16_Pin
- added J5: LCD, VapeRE:UNK_FPC_1x08-1MP_P0.5mm_Horizontal, symbol Connector_Generic_MountingPin:Conn_01x08_MountingPin
- added Q10: DTC114E, Package_TO_SOT_SMD:SOT-523, symbol Transistor_BJT:DTC114E
- added R22, R23, R24, R25, R26, R27, R28, R29, R30, R31, R32, R33, R34, R35, R36, R37, R38, R39, R40: 100, Resistor_SMD:R_0402_1005Metric, symbol Device:R_Small_US
- added R41: 511, Resistor_SMD:R_0402_1005Metric, symbol Device:R_Small_US
- added R42: 267, Resistor_SMD:R_0402_1005Metric, symbol Device:R_Small_US
- added R43: 330, Resistor_SMD:R_0402_1005Metric, symbol Device:R_Small_US
- added U10: LDO, Active:SOT95P230X117-3, symbol Connector_Generic:Conn_01x03
- U2: value RF01 -> BLueX Micro RF01 / BX2400
- U3: value ? -> PD64SH4AD
- U4: Topmark A7v47 -> A7y47
Connections:
- net +1V8: now reaches C10.1, C18.2, L1.1, U2.17 (VDD_1V8), U2.18 (VDD_DIG), U2.41 (VDD_VCO), U2.43 (VDD_CP), U2.44 (VDD_RF1), U2.47 (VDD_A)
- net BACKLIGHT: now reaches J1.9 (Pin_9), R7.2, TP1.1
- net P02 renamed ~{LCD_CS}
- net P03 renamed LED_BLU
- net P04 renamed ~{LCD_CLK}
- net P05 renamed LED_GRN
- net P06 renamed ~{LCD_DI}
- net P07 renamed ~{LCD_RST}
- net P09 renamed ~{LCD_DC}
- net P12 renamed LED_RED
- net P13 renamed LED_WH1
- net P21 renamed LED_WH2
- net P22 renamed LED_WHT
- new net: D13.1 (K), R31.1
- new net: Q10.3 (C), R22.2, R23.2, R24.2, R25.2, R26.2, R27.2, R28.2, R29.2, R30.2, R31.2, R32.2, R33.2, R34.2, R35.2, R36.2
- new net: D23.2 (RK), D24.2 (RK), D25.2 (RK), D26.2 (RK), R42.1
- new net: D23.3 (GK), D24.3 (GK), D25.3 (GK), D26.3 (GK), R43.1
- new net: D23.4 (BK), D24.4 (BK), D25.4 (BK), D26.4 (BK), R41.1
- new net: D10.1 (K), R28.1
- new net: D8.1 (K), R26.1
- new net: J10.11 (Pin_11), R37.1, R38.1
- new net: D19.1 (K), R37.2
- new net: D16.1 (K), R34.1
- new net: D4.1 (K), R22.1
- new net: D15.1 (K), R33.1
- new net: D14.1 (K), R32.1
- new net: D11.1 (K), R29.1
- new net: J10.10 (Pin_10), Q10.1 (B)
- new net: C21.2, C22.1, J10.7 (Pin_7), J10.8 (Pin_8), J5.2 (Pin_2), Q10.2 (E), U10.1 (Pin_1)
- new net: D20.1 (K), R38.2
- new net: J10.12 (Pin_12), R39.1, R40.1
- new net: D21.1 (K), R39.2
- new net: D22.1 (K), R40.2
- new net: D17.1 (K), R35.1
- new net: J10.1 (Pin_1), J5.8 (Pin_8)
- new net: J10.13 (Pin_13), R43.2
- new net: J10.14 (Pin_14), R42.2
- new net: J10.15 (Pin_15), R41.2
- new net: C21.1, J10.16 (Pin_16), U10.3 (Pin_3)
- new net: J10.2 (Pin_2), J5.7 (Pin_7)
- new net: J10.3 (Pin_3), J5.6 (Pin_6)
- new net: J10.4 (Pin_4), J5.5 (Pin_5)
- new net: J10.5 (Pin_5), J5.4 (Pin_4)
- new net: J10.6 (Pin_6), J5.3 (Pin_3)
- new net: J10.9 (Pin_9), J5.1 (Pin_1)
- new net: D18.1 (K), R36.1
- new net: D6.1 (K), R24.1
- new net: D7.1 (K), R25.1
- new net: D12.1 (K), R30.1
- new net: D5.1 (K), R23.1
- new net: D9.1 (K), R27.1
- new net 3V3: C22.2, D10.2 (A), D11.2 (A), D12.2 (A), D13.2 (A), D14.2 (A), D15.2 (A), D16.2 (A), D17.2 (A), D18.2 (A), D19.2 (A), D20.2 (A), D21.2 (A), D22.2 (A), D23.1 (A), D24.1 (A), D25.1 (A), D26.1 (A), D4.2 (A), D5.2 (A), D6.2 (A), D7.2 (A), D8.2 (A), D9.2 (A), U10.2 (Pin_2)
- no-connect marks 7 -> 8
Other:
- note added: "(SPIM0)"
- note added: "3V3"
- note added: "BACKLIGHT"
- note added: "CLK"
- note added: "D/C"
- note added: "DI"
- note added: "GND"
- note added: "TO LEDS"
- note added: "~{CS}"
- note added: "~{RST}"
- moved on the sheet: C1, C14, C15, C18, C2, C20, C3, C4, D3, J1, J2, J3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

Commit message: LDO regulator p/n
Parts:
- removed U4: LDO, Active:SOT95P230X117-3, symbol Connector_Generic:Conn_01x03
- added U4: CJ6330A33M, Active:SOT95P230X117-3, symbol Regulator_Linear:AP2127N3-1.2
- U5: value Conn_02x03_Counter_Clockwise -> Watchdog?; Topmark (none) -> 2402
Connections:
- net +3.3V: now also U4.2 (VO)
- net +BATT: now also U4.3 (VI)
- net GND: now also U4.1 (GND)
- net ~{RESET} renamed RESET
Other:
- moved on the sheet: C2, C3
