File: STW2915/STW2915.kicad_sch (KiCad schematic)
At the start: 62 parts, among them J1 USB_C_Receptacle_PowerOnly_6P, J2 LCD, Q1 SP1216, Q2 SP1216, Q3 Q_NMOS_GSD, Q4 Q_NMOS_GSD, Q5 Q_PMOS_GSD, Q6 Q_PMOS_GSD, SW2 SW_Push, U1 PY32F030K2, U2 LP4068, U3 PD64SH4BDPL2, U4 CJ6330A33M

Commit message: STW2915 tweaks
Parts:
- SW2: MPN (none) -> Xunpu TS-1077S-01526
- U3: value PD64SH4BDPL2 -> P25Q64SH; Topmark (none) -> PD64SH4BDPL2
Other:
- note added: "CURR asserts low to increase charge current to 2.2A for vaping while charging"
Changed lines of the file:
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@@
 	(generator_version "9.0")
 	(paper "A4")
+	(text "CURR asserts low\nto increase charge\ncurrent to 2.2A\nfor vaping while\ncharging"
+		(exclude_from_sim no)
+		(at 135.128 68.326 0)
+		(effects
+			(font
+				(size 1.27 1.27)
+			)
+		)
+	)
 	(junction
 		(at 265.43 34.29)
@@
 			)
 		)
-		(property "Value" "PD64SH4BDPL2"
+		(property "Value" "P25Q64SH"
 			(at 207.01 143.5099 0)
 			(effects
@@
 			)
 		)
+		(property "Topmark" "PD64SH4BDPL2"
+			(at 195.58 142.24 0)
+			(effects
+				(font
+					(size 1.27 1.27)
+				)
+				(hide yes)
+			)
+		)
 		(pin "6"
 		)
@@
 		(on_board yes)
 		(dnp no)
-		(fields_autoplaced yes)
 		(property "Reference" "SW2"
-			(at 55.88 172.72 0)
+			(at 56.134 169.672 0)
 			(effects
 				(font
@@
 		)
 		(property "Value" "SW_Push"
-			(at 55.88 175.26 0)
+			(at 56.134 172.212 0)
 			(effects
 				(font
@@
 			)
 		)
+		(property "MPN" "Xunpu TS-1077S-01526"
+			(at 64.262 175.006 0)
+			(effects
+				(font
+					(size 1.27 1.27)
+				)
+			)
+		)
